File: core/core.kicad_sch (KiCad schematic)
At the start: 49 parts, among them CN1 DF40C-100DS-0.4V, CN2 DF40C-100DS-0.4V, J1 Conn_01x02, J2 Conn_01x02, J3 Conn_01x03, J4 Conn_01x02, J5 Conn_01x02, J6 Conn_01x02, J7 Conn_01x02, U1 MCP73831T-2ACI/OT, U2 MAX17048G+T10, U3 TPS62840DLCR, U4 TLV70018DDCR, U5 TPS61023DRLR, U6 MAX98357A, U7 MAX98357A

Commit message: Add README, gitignore, banner
Parts:
- added C18: 100nF, symbol Device:C
- added C19: 1 µF, symbol Device:C
- added C20: 0.1 µF, symbol Device:C
- added FPC1: AFC01-S40FCA-00, luxera:FPC-SMD_AFC01-S40FCA-00, symbol luxera:AFC01-S40FCA-00
- added R12: 10k, symbol Device:R
- added SW1: SW_Push, symbol Switch:SW_Push
- added U8: IQS227B-00000000-TSR, luxera:SOT-23-6_L2.9-W1.6-P0.95-LS2.8-TL, symbol luxera:IQS227B-00000000-TSR
Connections:
- net +1V8: now also FPC1.24
- net +3V3: now also C20.1, FPC1.25, U8.5 (VDDHI)
- net CM4_3V3: now also R12.2
- net GND: now also CN2.79, CN2.80, CN2.85, CN2.86, CN2.91, CN2.92, C18.2, C19.2, C20.2, FPC1.1, FPC1.23, FPC1.34, FPC1.37, FPC1.4, FPC1.40, FPC1.9, SW1.2, U8.2 (GND)
- net SCL: now also FPC1.15, FPC1.31
- net SDA: now also FPC1.14, FPC1.30
- net SPK_L+: now also FPC1.28
- net VBAT: now also FPC1.26, FPC1.27
- net ToF_LPn: now reaches CN1.24
- net ToF_LPn: now also FPC1.17
- net PDM_DAT: now reaches CN1.28
- net PDM_DAT: now also FPC1.19
- net ToF_INT: now reaches CN1.30
- net ToF_INT: now also FPC1.16
- net PDM_CLK: now reaches CN1.31
- net PDM_CLK: now also FPC1.18
- net CAM_RST: now reaches CN1.34
- net CAM_RST: now also FPC1.11
- net AMB_INT: now reaches CN1.45
- net AMB_INT: now also FPC1.22
- net MCU_WAKE: now reaches CN1.46
- net MCU_WAKE: now also FPC1.32
- net SOM_IRQ: now reaches CN1.47
- net SOM_IRQ: now also FPC1.33
- net TOUCH_OUT: now reaches CN1.50
- net TOUCH_OUT: now also U8.1 (TOUT)
- net BTN: now reaches CN1.54
- net BTN: now also C18.1, R12.1, SW1.1
- net CAM_SCL: now reaches CN1.80
- net CAM_SCL: now also FPC1.36
- net CAM_SDA: now reaches CN1.82
- net CAM_SDA: now also FPC1.35
- net VPU_B: now reaches CN1.94
- net VPU_B: now also FPC1.21
- net VPU_A: now reaches CN1.96
- net VPU_A: now also FPC1.20
- net CAM_EN: now reaches CN1.97
- net CAM_EN: now also FPC1.12
- net CSI_D0N: now reaches CN2.15
- net CSI_D0N: now also FPC1.6
- net CSI_D0P: now reaches CN2.17
- net CSI_D0P: now also FPC1.5
- net CSI_D1N: now reaches CN2.21
- net CSI_D1N: now also FPC1.8
- net CSI_D1P: now reaches CN2.23
- net CSI_D1P: now also FPC1.7
- net CSI_CKN: now reaches CN2.27
- net CSI_CKN: now also FPC1.3
- net CSI_CKP: now reaches CN2.29
- net CSI_CKP: now also FPC1.2
- net DSI_D0N: now reaches CN2.75
- net DSI_D0P: now reaches CN2.77
- net DSI_D1N: now reaches CN2.81
- net DSI_D1P: now reaches CN2.83
- net DSI_CKN: now reaches CN2.87
- net DSI_CKP: now reaches CN2.89
- new net: C19.1, U8.4 (VREG)
- new net CAM_MCLK: FPC1.10
- new net CAM_PWR: FPC1.13
- new net SPK_L−: FPC1.29
- new net TOUCH_PAD: U8.6 (Cx)
- no-connect marks 7 -> 8
Other:
- moved on the sheet: C12, C13, C14, C15, C16, C17, CN1, CN2, D2, J3, J4, J5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

Commit message: zones + branding
Parts:
- C1, C14, C16, C2, C5, C6, C9: footprint (none) -> Capacitor_SMD:C_0603_1608Metric
- C10, C11, C12, C13: footprint (none) -> Capacitor_SMD:C_0805_2012Metric
- C15, C17, C18, C19, C20, C3, C4, C7, C8: footprint (none) -> Capacitor_SMD:C_0402_1005Metric
- D2: footprint (none) -> LED_SMD:LED_0603_1608Metric
- J1, J2, J6, J7: footprint (none) -> Connector_JST:JST_PH_B2B-PH-K_1x02_P2.00mm_Vertical
- J3: footprint (none) -> Connector_PinHeader_2.54mm:PinHeader_1x03_P2.54mm_Vertical
- J4, J5: footprint (none) -> Connector_PinHeader_2.54mm:PinHeader_1x02_P2.54mm_Vertical
- L1: footprint (none) -> Inductor_SMD:L_Taiyo-Yuden_NR-30xx
- L2: footprint (none) -> Inductor_SMD:L_Taiyo-Yuden_NR-40xx
- R1, R10, R11, R12, R2, R3, R4, R5, R6, R7, R8, R9: footprint (none) -> Resistor_SMD:R_0402_1005Metric
- SW1: footprint (none) -> Button_Switch_SMD:SW_SPST_PTS645Sx43SMTR92
Changed lines of the file:
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@@
 			)
 		)
-		(property "Footprint" ""
+		(property "Footprint" "Capacitor_SMD:C_0603_1608Metric"
 			(at 162.2552 114.3 0)
 			(hide yes)
@@
 			)
 		)
-		(property "Footprint" ""
+		(property "Footprint" "Resistor_SMD:R_0402_1005Metric"
 			(at 140.97 91.948 90)
 			(hide yes)
@@
 			)
 		)
-		(property "Footprint" ""
+		(property "Footprint" "Capacitor_SMD:C_0603_1608Metric"
 			(at 78.4352 104.14 0)
 			(hide yes)
@@
 			)
 		)
-		(property "Footprint" ""
+		(property "Footprint" "Connector_PinHeader_2.54mm:PinHeader_1x02_P2.54mm_Vertical"
 			(at 321.31 54.61 0)
 			(hide yes)
@@
 			)
 		)
-		(property "Footprint" ""
+		(property "Footprint" "Connector_JST:JST_PH_B2B-PH-K_1x02_P2.00mm_Vertical"
 			(at 29.21 76.2 0)
 			(hide yes)
@@
 			)
 		)
-		(property "Footprint" ""
+		(property "Footprint" "Capacitor_SMD:C_0402_1005Metric"
 			(at 285.75 241.6048 0)
 			(hide yes)
@@
 			)
 		)
-		(property "Footprint" ""
+		(property "Footprint" "Capacitor_SMD:C_0603_1608Metric"
 			(at 199.39 180.6448 0)
 			(hide yes)
@@
 			)
 		)
-		(property "Footprint" ""
+		(property "Footprint" "Resistor_SMD:R_0402_1005Metric"
 			(at 242.57 102.108 90)
 			(hide yes)
@@
 			)
 		)
-		(property "Footprint" ""
+		(property "Footprint" "Capacitor_SMD:C_0402_1005Metric"
 			(at 209.2452 82.55 0)
 			(hide yes)
@@
 			)
 		)
-		(property "Footprint" ""
+		(property "Footprint" "Resistor_SMD:R_0402_1005Metric"
 			(at 242.57 110.998 90)
 			(hide yes)
@@
 			)
 		)
-		(property "Footprint" ""
+		(property "Footprint" "Resistor_SMD:R_0402_1005Metric"
 			(at 204.47 237.998 90)
 			(hide yes)
@@
 			)
 		)
-		(property "Footprint" ""
+		(property "Footprint" "Inductor_SMD:L_Taiyo-Yuden_NR-30xx"
 			(at 66.04 43.18 0)
 			(hide yes)
@@
 			)
 		)
-		(property "Footprint" ""
+		(property "Footprint" "Resistor_SMD:R_0402_1005Metric"
 			(at 126.492 34.29 90)
 			(hide yes)
@@
 			)
 		)
-		(property "Footprint" ""
+		(property "Footprint" "Connector_JST:JST_PH_B2B-PH-K_1x02_P2.00mm_Vertical"
 			(at 29.21 85.09 0)
 			(hide yes)
@@
 			)
 		)
-		(property "Footprint" ""
+		(property "Footprint" "Capacitor_SMD:C_0402_1005Metric"
 			(at 217.17 23.1648 0)
 			(hide yes)
@@
 			)
 		)
-		(property "Footprint" ""
+		(property "Footprint" "Capacitor_SMD:C_0603_1608Metric"
 			(at 53.34 59.9948 0)
 			(hide yes)
@@
 			)
 		)
-		(property "Footprint" ""
+		(property "Footprint" "Capacitor_SMD:C_0402_1005Metric"
 			(at 208.28 245.4148 0)
 			(hide yes)
@@
 			)
 		)
-		(property "Footprint" ""
+		(property "Footprint" "Capacitor_SMD:C_0805_2012Metric"
 			(at 166.37 25.7048 0)
 			(hide yes)
@@
 			)
 		)
-		(property "Footprint" ""
+		(property "Footprint" "Capacitor_SMD:C_0603_1608Metric"
 			(at 313.69 185.7248 0)
 			(hide yes)
@@
 			)
 		)
-		(property "Footprint" ""
+		(property "Footprint" "Connector_JST:JST_PH_B2B-PH-K_1x02_P2.00mm_Vertical"
 			(at 391.16 195.58 0)
 			(hide yes)
@@
 			)
 		)
-		(property "Footprint" ""
+		(property "Footprint" "Capacitor_SMD:C_0402_1005Metric"
 			(at 313.69 198.4248 0)
 			(hide yes)
@@
 			)
 		)
-		(property "Footprint" ""
+		(property "Footprint" "Button_Switch_SMD:SW_SPST_PTS645Sx43SMTR92"
 			(at 204.47 219.71 0)
 			(hide yes)
@@
 			)
 		)
-		(property "Footprint" ""
+		(property "Footprint" "Capacitor_SMD:C_0402_1005Metric"
 			(at 209.55 50.4952 0)
 			(hide yes)
@@
 			)
 		)
-		(property "Footprint" ""
+		(property "Footprint" "Capacitor_SMD:C_0805_2012Metric"
 			(at 334.01 71.4248 0)
 			(hide yes)
@@
 			)
 		)
-		(property "Footprint" ""
+		(property "Footprint" "Resistor_SMD:R_0402_1005Metric"
 			(at 139.7 76.708 90)
 			(hide yes)
@@
 			)
 		)
-		(property "Footprint" ""
+		(property "Footprint" "Connector_PinHeader_2.54mm:PinHeader_1x03_P2.54mm_Vertical"
 			(at 321.31 34.29 0)
 			(hide yes)
@@
 			)
 		)
-		(property "Footprint" ""
+		(property "Footprint" "Capacitor_SMD:C_0805_2012Metric"
 			(at 173.99 35.8648 0)
 			(hide yes)
@@
 			)
 		)
-		(property "Footprint" ""
+		(property "Footprint" "Resistor_SMD:R_0402_1005Metric"
 			(at 83.82 50.038 90)
 			(hide yes)
@@
 			)
 		)
-		(property "Footprint" ""
+		(property "Footprint" "Resistor_SMD:R_0402_1005Metric"
 			(at 115.062 34.29 90)
 			(hide yes)
@@
 			)
 		)
-		(property "Footprint" ""
+		(property "Footprint" "Capacitor_SMD:C_0402_1005Metric"
 			(at 174.9552 114.3 0)
 			(hide yes)
@@
 			)
 		)
-		(property "Footprint" ""
+		(property "Footprint" "Resistor_SMD:R_0402_1005Metric"
 			(at 224.79 203.962 90)
 			(hide yes)
@@
 			)
 		)
-		(property "Footprint" ""
+		(property "Footprint" "Inductor_SMD:L_Taiyo-Yuden_NR-40xx"
 			(at 163.83 48.26 0)
 			(hide yes)
@@
 			)
 		)
-		(property "Footprint" ""
+		(property "Footprint" "Capacitor_SMD:C_0603_1608Metric"
 			(at 110.1852 50.8 0)
 			(hide yes)
@@
 			)
 		)
-		(property "Footprint" ""
+		(property "Footprint" "Resistor_SMD:R_0402_1005Metric"
 			(at 242.57 121.158 90)
 			(hide yes)
@@
 			)
 		)
-		(property "Footprint" ""
+		(property "Footprint" "Capacitor_SMD:C_0402_1005Metric"
 			(at 199.39 193.3448 0)
 			(hide yes)
@@
 			)
 		)
-		(property "Footprint" ""
+		(property "Footprint" "LED_SMD:LED_0603_1608Metric"
 			(at 370.84 49.53 0)
 			(hide yes)
@@
 			)
 		)
-		(property "Footprint" ""
+		(property "Footprint" "Capacitor_SMD:C_0805_2012Metric"
 			(at 334.01 81.5848 0)
 			(hide yes)
@@
 			)
 		)
-		(property "Footprint" ""
+		(property "Footprint" "Connector_PinHeader_2.54mm:PinHeader_1x02_P2.54mm_Vertical"
 			(at 321.31 45.72 0)
 			(hide yes)
@@
 			)
 		)
-		(property "Footprint" ""
+		(property "Footprint" "Resistor_SMD:R_0402_1005Metric"
 			(at 363.22 51.308 90)
 			(hide yes)
@@
 			)
 		)
-		(property "Footprint" ""
+		(property "Footprint" "Connector_JST:JST_PH_B2B-PH-K_1x02_P2.00mm_Vertical"
 			(at 276.86 190.5 0)
 			(hide yes)
@@
 			)
 		)
-		(property "Footprint" ""
+		(property "Footprint" "Capacitor_SMD:C_0402_1005Metric"
 			(at 293.6748 222.25 0)
 			(hide yes)
@@
 			)
 		)
-		(property "Footprint" ""
+		(property "Footprint" "Resistor_SMD:R_0402_1005Metric"
 			(at 93.98 81.788 90)
 			(hide yes)
@@
 			)
 		)
-		(property "Footprint" ""
+		(property "Footprint" "Capacitor_SMD:C_0603_1608Metric"
 			(at 27.6352 38.1 0)
 			(hide yes)
